File: KiCad/Controller_v4.3/Controller_v4.3.kicad_pcb (KiCad board)
At the start: 2 copper layers, 82.7 x 72.9 mm, 47 parts, among them J1 Barrel_Jack_Switch, J2 USB_C_Receptacle_USB2.0_16P, J3 Conn_02x03_Odd_Even, Q1 MMBT3904, Q2 MMBT3904, Q3 BC857, Q4 Q_PMOS_GDS, Q5 BC857, U1 CH340C, U2 ESP32-WROOM-32E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

Commit message: Relabeled Components
Parts:
- renumbered C9 to C1, C11 to C10, C4 to C11, C3 to C12, C10 to C2, C6 to C3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
