File: KiCad/Controller_v4.3/Controller_v4.3.kicad_pcb (KiCad board)
At the start: 2 copper layers, 82.7 x 72.9 mm, 47 parts, among them J1 USB_C_Receptacle_USB2.0_16P, J2 Barrel_Jack_Switch, J3 Conn_02x03_Odd_Even, Q1 Q_PMOS_GDS, Q2 BC857, Q3 BC857, Q4 MMBT3904, Q5 MMBT3904, U1 AMS1117-3.3, U2 ESP32-WROOM-32E, U3 AP63205WU, U4 SN74LVC1T45DBV, U5 CH340C

Commit message: Consolidate controller bom
Parts:
- added SYM1: ~, rt_Logo:RT_Logo_10mm_Silkscreen, B.Cu at (112.6, 110.4)
- C1: value 470u -> 470u 25V
- C4: value 100n -> 10u
