File: KiCad/Controller_v4.3/Controller_v4.3.kicad_sch (KiCad schematic)
At the start: 47 parts, among them J1 USB_C_Receptacle_USB2.0_16P, J2 Barrel_Jack_Switch, J3 Conn_02x03_Odd_Even, Q1 Q_PMOS_GDS, Q2 BC857, Q3 BC857, Q4 MMBT3904, Q5 MMBT3904, U1 AMS1117-3.3, U2 ESP32-WROOM-32E, U3 AP63205WU, U4 SN74LVC1T45DBV, U5 CH340C

Commit message: Consolidate controller bom
Parts:
- added SYM1: (no value), rt_Logo:RT_Logo_10mm_Silkscreen, symbol rt_Logo:RT_Logo
- C1: value 470u -> 470u 25V; Part Number (none) -> EEE-FK1E471AP
- C11, C12: Part Number (none) -> CL31B226MPHNNNE
- C4: value 100n -> 10u; Part Number (none) -> CL31B106KAHNNNE
- C6: Part Number (none) -> CL31B106KAHNNNE
- J1: Part Number (none) -> USB4105-GF-A-120
